File: Led_Controller.sch (KiCad schematic (older format))
At the start: 12 parts, among them U3 ADP162AUJZ-3.3, U4 STM32L151CBT6-A

Commit message: Update Led_Controller.sch
Parts:
- C10, C11, C12, C13, C14, C15, C16, C17, C18: symbol CP -> Device:CP
- STRIP2: symbol STRIP_8P -> TCKB:STRIP_8P
- U3: symbol ADP162AUJZ-3.3 -> TCKB:ADP162AUJZ-3.3
- U4: symbol STM32L053C8 -> TCKB:STM32L053C8
Connections:
- wire segments 99 -> 119
Changed lines of the file:
@@
-EESchema Schematic File Version 2
-LIBS:power
-LIBS:device
-LIBS:transistors
-LIBS:conn
-LIBS:linear
-LIBS:regul
-LIBS:74xx
-LIBS:cmos4000
-LIBS:adc-dac
-LIBS:memory
-LIBS:xilinx
-LIBS:microcontrollers
-LIBS:dsp
-LIBS:microchip
-LIBS:analog_switches
-LIBS:motorola
-LIBS:texas
-LIBS:intel
-LIBS:audio
-LIBS:interface
-LIBS:digital-audio
-LIBS:philips
-LIBS:display
-LIBS:cypress
-LIBS:siliconi
-LIBS:opto
-LIBS:atmel
-LIBS:contrib
-LIBS:valves
-LIBS:TCKB
-LIBS:TCKB-cache
-EELAYER 25 0
+EESchema Schematic File Version 4
+EELAYER 30 0
 EELAYER END
 $Descr A4 11693 8268
@@
 $EndDescr
 $Comp
-L GNDPWR #PWR019
+L TCKB-rescue:GNDPWR #PWR019
 U 1 1 5663605A
 P 6850 4900
+AR Path="/5663605A" Ref="#PWR019"  Part="1"
+AR Path="/56632A89/5663605A" Ref="#PWR019"  Part="1"
 F 0 "#PWR019" H 6850 4700 50  0001 C CNN
 F 1 "GNDPWR" H 6850 4770 50  0000 C CNN
@@
 	6400 4750 6400 4800
 Wire Wire Line
-	6400 4800 7000 4800
+	6400 4800 6550 4800
 Wire Wire Line
 	7000 4800 7000 4750
@@
 Connection ~ 6700 4800
 $Comp
-L CP C14
+L Device:CP C14
 U 1 1 5663606A
 P 9850 1050
@@
 $EndComp
 $Comp
-L GNDPWR #PWR020
+L TCKB-rescue:GNDPWR #PWR020
 U 1 1 56636077
 P 9650 1300
+AR Path="/56636077" Ref="#PWR020"  Part="1"
+AR Path="/56632A89/56636077" Ref="#PWR020"  Part="1"
 F 0 "#PWR020" H 9650 1100 50  0001 C CNN
 F 1 "GNDPWR" H 9650 1170 50  0000 C CNN
@@
 	6400 1250 6400 1200
 Wire Wire Line
-	6400 1200 7000 1200
+	6400 1200 6550 1200
 Wire Wire Line
 	7000 1200 7000 1250
@@
 Connection ~ 6550 1200
 $Comp
-L STM32L053C8 U4
+L TCKB:STM32L053C8 U4
 U 1 1 566360B1
 P 6700 3000
@@
 STM32 Coupling
 $Comp
-L CP C15
+L Device:CP C15
 U 1 1 566360BE
 P 10150 1050
@@
 $EndComp
 $Comp
-L CP C17
+L Device:CP C17
 U 1 1 566360C5
 P 10750 1050
@@
 $EndComp
 $Comp
-L CP C16
+L Device:CP C16
 U 1 1 566360D3
 P 10450 1050
@@
 NoConn ~ 5200 2300
 Wire Wire Line
-	9650 850  10750 850
+	9650 850  9850 850
 Wire Wire Line
 	10750 850  10750 900
 Wire Wire Line
-	9650 1250 10750 1250
+	9650 1250 9850 1250
 Wire Wire Line
 	10750 1250 10750 1200
@@
 	4850 1750 5200 1750
 $Comp
-L GNDPWR #PWR021
+L TCKB-rescue:GNDPWR #PWR021
 U 1 1 5663C587
 P 5600 7350
+AR Path="/5663C587" Ref="#PWR021"  Part="1"
+AR Path="/56632A89/5663C587" Ref="#PWR021"  Part="1"
 F 0 "#PWR021" H 5600 7150 50  0001 C CNN
 F 1 "GNDPWR" H 5600 7220 50  0000 C CNN
@@
 $EndComp
 $Comp
-L CP C13
+L Device:CP C13
 U 1 1 5663C58D
 P 6450 7100
@@
 $EndComp
 $Comp
-L +5V #PWR022
+L power:+5V #PWR022
 U 1 1 5663C594
 P 4750 6700
@@
 $EndComp
 $Comp
-L CP C12
+L Device:CP C12
 U 1 1 5663C59A
 P 6200 7100
@@
 $EndComp
 $Comp
-L CP C10
+L Device:CP C10
 U 1 1 5663C5A1
 P 4750 7100
@@
 $EndComp
 $Comp
-L CP C11
+L Device:CP C11
 U 1 1 5663C5A8
 P 5000 7100
@@
 $EndComp
 Wire Wire Line
-	4750 6700 4750 6950
-Wire Wire Line
-	4750 6900 5150 6900
+	4750 6700 4750 6750
+Wire Wire Line
+	4750 6900 5000 6900
 Connection ~ 4750 6900
 Wire Wire Line
@@
 	5600 7350 5600 7100
 $Comp
-L GNDPWR #PWR023
+L TCKB-rescue:GNDPWR #PWR023
 U 1 1 5663C5BA
 P 4750 7350
+AR Path="/5663C5BA" Ref="#PWR023"  Part="1"
+AR Path="/56632A89/5663C5BA" Ref="#PWR023"  Part="1"
 F 0 "#PWR023" H 4750 7150 50  0001 C CNN
 F 1 "GNDPWR" H 4750 7220 50  0000 C CNN
@@
 $EndComp
 $Comp
-L GNDPWR #PWR024
+L TCKB-rescue:GNDPWR #PWR024
 U 1 1 5663C5C0
 P 6450 7350
+AR Path="/5663C5C0" Ref="#PWR024"  Part="1"
+AR Path="/56632A89/5663C5C0" Ref="#PWR024"  Part="1"
 F 0 "#PWR024" H 6450 7150 50  0001 C CNN
 F 1 "GNDPWR" H 6450 7220 50  0000 C CNN
@@
 $EndComp
 Wire Wire Line
-	4750 7250 4750 7350
+	4750 7250 4750 7300
 Wire Wire Line
 	5000 7250 5000 7300
@@
 Connection ~ 4750 7300
 Wire Wire Line
-	6450 7250 6450 7350
+	6450 7250 6450 7300
 Wire Wire Line
 	6200 7250 6200 7300
@@
 NoConn ~ 6050 6900
 $Comp
-L ADP162AUJZ-3.3 U3
+L TCKB:ADP162AUJZ-3.3 U3
 U 1 1 5663C5D1
 P 5600 6800
@@
 	2900 4900 3050 4900
 $Comp
-L +3V3_AUX #PWR025
+L TCKB:+3V3_AUX #PWR025
 U 1 1 57F41FFA
 P 6450 6700
@@
 $EndComp
 Wire Wire Line
-	6050 6750 6450 6750
-Wire Wire Line
-	6450 6700 6450 6950
+	6050 6750 6200 6750
+Wire Wire Line
+	6450 6700 6450 6750
 Connection ~ 6200 6750
 Connection ~ 6450 6750
 $Comp
-L +3V3_AUX #PWR026
+L TCKB:+3V3_AUX #PWR026
 U 1 1 57F42CF9
 P 6850 1100
@@
 Connection ~ 6850 1200
 $Comp
-L +3V3_AUX #PWR027
+L TCKB:+3V3_AUX #PWR027
 U 1 1 57F43B08
 P 9650 800
@@
 	9650 800  9650 850
 $Comp
-L +3V3_AUX #PWR028
+L TCKB:+3V3_AUX #PWR028
 U 1 1 57F44909
 P 9600 5100
@@
 SWO_2
 $Comp
-L CP C18
+L Device:CP C18
 U 1 1 57F817C3
 P 9200 5750
@@
 $EndComp
 $Comp
-L STRIP_8P STRIP2
+L TCKB:STRIP_8P STRIP2
 U 1 1 57F817CE
 P 10300 5100
@@
 $EndComp
 $Comp
-L GNDPWR #PWR029
+L TCKB-rescue:GNDPWR #PWR029
 U 1 1 57F908DC
 P 10200 5600
+AR Path="/57F908DC" Ref="#PWR029"  Part="1"
+AR Path="/56632A89/57F908DC" Ref="#PWR029"  Part="1"
 F 0 "#PWR029" H 10200 5400 50  0001 C CNN
 F 1 "GNDPWR" V 10200 5350 50  0000 C CNN
@@
 	10300 5200 10050 5200
 $Comp
-L GNDPWR #PWR030
+L TCKB-rescue:GNDPWR #PWR030
 U 1 1 57F908EE
 P 9200 5950
+AR Path="/57F908EE" Ref="#PWR030"  Part="1"
+AR Path="/56632A89/57F908EE" Ref="#PWR030"  Part="1"
 F 0 "#PWR030" H 9200 5750 50  0001 C CNN
 F 1 "GNDPWR" H 9200 5820 50  0000 C CNN
@@
 Bootloader
 Wire Wire Line
-	8900 5500 10300 5500
+	8900 5500 9200 5500
 Wire Wire Line
 	10050 5700 10300 5700
@@
 NoConn ~ 8200 1750
 NoConn ~ 8200 1850
+Wire Wire Line
+	6550 4800 6700 4800
+Wire Wire Line
+	6700 4800 6850 4800
+Wire Wire Line
+	6700 1200 6850 1200
+Wire Wire Line
+	6550 1200 6700 1200
+Wire Wire Line
+	10450 1250 10750 1250
+Wire Wire Line
+	10150 1250 10450 1250
+Wire Wire Line
+	9850 1250 10150 1250
+Wire Wire Line
+	9850 850  10150 850
+Wire Wire Line
+	10150 850  10450 850
+Wire Wire Line
+	10450 850  10750 850
+Wire Wire Line
+	4750 6900 4750 6950
+Wire Wire Line
+	4750 6750 4750 6900
+Wire Wire Line
+	5000 6900 5150 6900
+Wire Wire Line
+	4750 7300 4750 7350
+Wire Wire Line
+	6450 7300 6450 7350
+Wire Wire Line
+	6200 6750 6450 6750
+Wire Wire Line
+	6450 6750 6450 6950
+Wire Wire Line
+	6850 1200 7000 1200
+Wire Wire Line
+	9200 5500 10300 5500
+Wire Wire Line
+	6850 4800 7000 4800
 $EndSCHEMATC
