File: Led_Matrix.sch (KiCad schematic (older format))
At the start: 102 parts, among them Q1 FDN359BN, Q10 BSS84P, Q11 BSS84P, Q12 BSS84P, Q13 BSS84P, Q14 BSS84P, Q15 BSS84P, Q16 BSS84P, Q17 BSS84P, Q18 BSS84P, Q19 BSS84P, Q2 FDN359BN, Q3 FDN359BN, Q4 FDN359BN, Q5 FDN359BN, Q6 BSS84P, Q7 BSS84P, Q8 BSS84P, Q9 BSS84P

Commit message: Update Led_Matrix.sch
Parts:
- LED1, LED10, LED11, LED12, LED13, LED14, LED15, LED16, LED17, LED18, LED19, LED2, LED20, LED21, LED22, LED23, LED24, LED25, LED26, LED27, LED28, LED29, LED3, LED30, LED31, LED32, LED33, LED34, LED35, LED36, LED37, LED38, LED39, LED4, LED40, LED41, LED42, LED43, LED44, LED45, LED46, LED47, LED48, LED49, LED5, LED50, LED51, LED52, LED53, LED54, LED55, LED56, LED57, LED58, LED59, LED6, LED60, LED61, LED62, LED63, LED64, LED7, LED8, LED9: symbol LED -> TCKB-rescue:LED
- Q1, Q2, Q3, Q4, Q5: symbol FDN359BN -> TCKB:FDN359BN
- Q10, Q11, Q12, Q13, Q14, Q15, Q16, Q17, Q18, Q19, Q6, Q7, Q8, Q9: symbol BSS84P -> TCKB:BSS84P
- R10, R11, R12, R13, R14, R15, R16, R17, R19, R21, R23, R25, R27, R29, R31, R33, R7, R8, R9: symbol R -> Device:R
Connections:
- wire segments 254 -> 391
