File: Matrix.sch (KiCad schematic (older format))
At the start: 134 parts, among them SW10 k_7, SW11 k_8, SW12 k_9, SW13 k_0, SW14 k_MINUS, SW15 k_EQUAL, SW16 k_BSPACE, SW17 k_TAB, SW18 k_Q, SW19 k_W, SW20 k_E, SW21 k_R, SW22 k_T, SW23 k_Y, SW24 k_U, SW25 k_I, SW26 k_O, SW27 k_P, SW28 k_LBRACKET, SW29 k__RBRACKET, SW3 k_ESC, SW30 k_BSLASH_ANSI, SW31 k_CAPSLOCK, SW32 k_A, SW33 k_S, SW34 k_D, SW35 k_F, SW36 k_G, SW37 k_H, SW38 k_J, SW39 k_K, SW4 k_1, SW40 k_L, SW41 k_SEMICOLON, SW42 k_QUOTE, SW43 k_BSLASH_ISO, SW44 k_ENTER_ISO, SW45 k_ENTER_ANSI, SW46 k_LSHIFT_ISO, SW47 k_NU_BSLASH_ISO, SW48 k_Z, SW49 k_X, SW5 k_2, SW50 k_C, SW51 k_V, SW52 k_B, SW53 k_N, SW54 k_M, SW55 k_COMMA, SW56 k_DOT, SW57 k_SLASH, SW58 k_RSHIFT, SW59 k_LSHIFT_ANSI, SW6 k_3, SW60 k_LCTRL, SW61 k_LGUI, SW62 k_LALT, SW63 k_SPACE, SW64 k_RALT, SW65 k_RGUI, SW66 k_RMENU, SW67 k_RCTRL, SW7 k_4, SW8 k_5, SW9 k_6

Commit message: Update Matrix.sch
Parts:
- D10, D11, D12, D13, D14, D15, D16, D17, D18, D19, D20, D21, D22, D23, D24, D25, D26, D27, D28, D29, D3, D30, D31, D32, D33, D34, D35, D36, D37, D38, D39, D4, D40, D41, D42, D43, D44, D45, D46, D47, D48, D49, D5, D50, D51, D52, D53, D54, D55, D56, D57, D58, D59, D6, D60, D61, D62, D63, D64, D65, D7, D8, D9: symbol D -> Device:D
- ST1, ST2, ST3, ST4, ST5, ST6: symbol Cherry_Stab -> TCKB:Cherry_Stab
- SW10, SW11, SW12, SW13, SW14, SW15, SW16, SW17, SW18, SW19, SW20, SW21, SW22, SW23, SW24, SW25, SW26, SW27, SW28, SW29, SW3, SW30, SW31, SW32, SW33, SW34, SW35, SW36, SW37, SW38, SW39, SW4, SW40, SW41, SW42, SW43, SW44, SW45, SW46, SW47, SW48, SW49, SW5, SW50, SW51, SW52, SW53, SW54, SW55, SW56, SW57, SW58, SW59, SW6, SW60, SW61, SW62, SW63, SW64, SW65, SW66, SW67, SW7, SW8, SW9: symbol MX -> TCKB:MX
Connections:
- wire segments 271 -> 387
