File: TCKB.sch (KiCad schematic (older format))
At the start: 20 parts, among them P1 Mini_USB, SW1 DIP4P, U1 STM32L053C8T6, U2 ADP162AUJZ-3.3

Commit message: Update TCKB.sch
Parts:
- C1, C2, C3, C4, C5, C6, C7, C8, C9: symbol CP -> Device:CP
- D2: symbol LED -> TCKB-rescue:LED
- P1: symbol Mini_USB -> TCKB:Mini_USB
- R1, R2, R3, R5, R6: symbol R -> Device:R
- STRIP1: symbol STRIP_8P -> TCKB:STRIP_8P
- SW1: symbol DIP4P -> TCKB:DIP4P
- U1: symbol STM32L053C8 -> TCKB:STM32L053C8
- U2: symbol ADP162AUJZ-3.3 -> TCKB:ADP162AUJZ-3.3
Connections:
- wire segments 128 -> 157
Changed lines of the file:
@@
-EESchema Schematic File Version 2
-LIBS:power
-LIBS:device
-LIBS:transistors
-LIBS:conn
-LIBS:linear
-LIBS:regul
-LIBS:74xx
-LIBS:cmos4000
-LIBS:adc-dac
-LIBS:memory
-LIBS:xilinx
-LIBS:microcontrollers
-LIBS:dsp
-LIBS:microchip
-LIBS:analog_switches
-LIBS:motorola
-LIBS:texas
-LIBS:intel
-LIBS:audio
-LIBS:interface
-LIBS:digital-audio
-LIBS:philips
-LIBS:display
-LIBS:cypress
-LIBS:siliconi
-LIBS:opto
-LIBS:atmel
-LIBS:contrib
-LIBS:valves
-LIBS:TCKB
-LIBS:TCKB-cache
-EELAYER 25 0
+EESchema Schematic File Version 4
+EELAYER 30 0
 EELAYER END
 $Descr A4 11693 8268
@@
 $EndDescr
 $Comp
-L DIP4P SW1
+L TCKB:DIP4P SW1
 U 1 1 56425467
 P 1550 1550
@@
 $EndComp
 $Comp
-L +3V3 #PWR01
+L power:+3V3 #PWR01
 U 1 1 56425B3A
 P 5800 6750
@@
 $EndComp
 $Comp
-L +5V #PWR02
+L power:+5V #PWR02
 U 1 1 56425B76
 P 8950 2350
@@
 $EndComp
 $Comp
-L GNDPWR #PWR03
+L TCKB-rescue:GNDPWR #PWR03
 U 1 1 56425B9E
 P 8950 3400
@@
 NoConn ~ 8950 2900
 $Comp
-L GNDPWR #PWR04
+L TCKB-rescue:GNDPWR #PWR04
 U 1 1 56425FFD
 P 5950 4750
@@
 	5500 4600 5500 4650
 Wire Wire Line
-	5500 4650 6100 4650
+	5500 4650 5650 4650
 Wire Wire Line
 	6100 4650 6100 4600
@@
 Connection ~ 5800 4650
 $Comp
-L CP C2
+L Device:CP C2
 U 1 1 56426378
 P 9800 1050
@@
 $EndComp
 $Comp
-L +3V3 #PWR05
+L power:+3V3 #PWR05
 U 1 1 564263A2
 P 9600 800
@@
 $EndComp
 $Comp
-L GNDPWR #PWR06
+L TCKB-rescue:GNDPWR #PWR06
 U 1 1 564263C6
 P 9600 1300
@@
 	9600 1300 9600 1250
 $Comp
-L GNDPWR #PWR07
+L TCKB-rescue:GNDPWR #PWR07
 U 1 1 56427188
 P 10450 5700
@@
 $EndComp
 $Comp
-L +3V3 #PWR08
+L power:+3V3 #PWR08
 U 1 1 564271BD
 P 9850 5200
@@
 	7500 3000 7300 3000
 $Comp
-L R R1
+L Device:R R1
 U 1 1 56429B59
 P 2550 1300
@@
 $EndComp
 $Comp
-L GNDPWR #PWR09
+L TCKB-rescue:GNDPWR #PWR09
 U 1 1 56429D89
 P 4950 7400
@@
 $EndComp
 $Comp
-L GNDPWR #PWR010
+L TCKB-rescue:GNDPWR #PWR010
 U 1 1 56429E90
 P 2550 1500
@@
 $EndComp
 $Comp
-L +3V3 #PWR011
+L power:+3V3 #PWR011
 U 1 1 56429EF1
 P 5950 950
@@
 $EndComp
 $Comp
-L GNDPWR #PWR012
+L TCKB-rescue:GNDPWR #PWR012
 U 1 1 56429EF8
 P 9450 6050
@@
 	5500 1100 5500 1050
 Wire Wire Line
-	5500 1050 6100 1050
+	5500 1050 5650 1050
 Wire Wire Line
 	6100 1050 6100 1100
@@
 Connection ~ 5650 1050
 $Comp
-L LED D2
+L TCKB-rescue:LED D2
 U 1 1 56430F38
 P 10350 2950
@@
 	10350 2750 10350 2650
 $Comp
-L +5V #PWR013
+L power:+5V #PWR013
 U 1 1 56433EA7
 P 10350 2250
@@
 $EndComp
 $Comp
-L STM32L053C8 U1
+L TCKB:STM32L053C8 U1
 U 1 1 56439253
 P 5800 2850
@@
 	7300 2800 8450 2800
 $Comp
-L CP C9
+L Device:CP C9
 U 1 1 564701EB
 P 5800 7150
@@
 $EndComp
 $Comp
-L +5V #PWR014
+L power:+5V #PWR014
 U 1 1 564709E3
 P 4100 6750
@@
 $EndComp
 $Comp
-L CP C8
+L Device:CP C8
 U 1 1 5647163C
 P 5550 7150
@@
 $EndComp
 $Comp
-L CP C6
+L Device:CP C6
 U 1 1 564716AD
 P 4100 7150
@@
 $EndComp
 $Comp
-L CP C7
+L Device:CP C7
 U 1 1 564716B3
 P 4350 7150
@@
 $EndComp
 Wire Wire Line
-	4100 6750 4100 7000
-Wire Wire Line
-	4100 6950 4500 6950
+	4100 6750 4100 6800
+Wire Wire Line
+	4100 6950 4350 6950
 Connection ~ 4100 6950
 Wire Wire Line
@@
 Connection ~ 4350 6950
 Wire Wire Line
-	5800 6750 5800 7000
-Wire Wire Line
-	5400 6800 5800 6800
+	5800 6750 5800 6800
+Wire Wire Line
+	5400 6800 5550 6800
 Connection ~ 5800 6800
 Wire Wire Line
 	4950 7400 4950 7150
 $Comp
-L GNDPWR #PWR015
+L TCKB-rescue:GNDPWR #PWR015
 U 1 1 5647249B
 P 4100 7400
@@
 $EndComp
 $Comp
-L GNDPWR #PWR016
+L TCKB-rescue:GNDPWR #PWR016
 U 1 1 564724F2
 P 5800 7400
@@
 $EndComp
 Wire Wire Line
-	4100 7300 4100 7400
+	4100 7300 4100 7350
 Wire Wire Line
 	4350 7300 4350 7350
@@
 Connection ~ 4100 7350
 Wire Wire Line
-	5800 7300 5800 7400
+	5800 7300 5800 7350
 Wire Wire Line
 	5550 7300 5550 7350
@@
 NoConn ~ 5400 6950
 $Comp
-L ADP162AUJZ-3.3 U2
+L TCKB:ADP162AUJZ-3.3 U2
 U 1 1 56472B9E
 P 4950 6850
@@
 $EndComp
 $Comp
-L CP C3
+L Device:CP C3
 U 1 1 56477E1E
 P 10100 1050
@@
 $EndComp
 $Comp
-L CP C5
+L Device:CP C5
 U 1 1 56477E8E
 P 10700 1050
@@
 $EndComp
 $Comp
-L CP C1
+L Device:CP C1
 U 1 1 56477E94
 P 9450 5850
@@
 $EndComp
 $Comp
-L CP C4
+L Device:CP C4
 U 1 1 56477F0C
 P 10400 1050
@@
 NoConn ~ 4300 2150
 Wire Wire Line
-	9600 850  10700 850
+	9600 850  9800 850
 Wire Wire Line
 	10700 850  10700 900
 Wire Wire Line
-	9600 1250 10700 1250
+	9600 1250 9800 1250
 Wire Wire Line
 	10700 1250 10700 1200
@@
 Connection ~ 10400 850
 $Comp
-L Mini_USB P1
+L TCKB:Mini_USB P1
 U 1 1 564780D8
 P 8950 2600
@@
 $EndComp
 Wire Wire Line
-	8950 3000 8950 3400
+	8950 3000 8950 3350
 Wire Wire Line
 	9200 3300 9200 3350
 Wire Wire Line
-	8950 3350 9500 3350
+	8950 3350 9200 3350
 Connection ~ 8950 3350
 Wire Wire Line
@@
 	7550 2600 7300 2600
 $Comp
-L R R5
+L Device:R R5
 U 1 1 564A01EE
 P 10350 2500
@@
 $EndComp
 $Comp
-L R R2
+L Device:R R2
 U 1 1 564A2941
 P 8600 2700
@@
 $EndComp
 $Comp
-L R R3
+L Device:R R3
 U 1 1 564A316D
 P 8600 2800
@@
 	8200 2100 7300 2100
 Wire Wire Line
-	7300 2200 8200 2200
+	7300 2200 8100 2200
 Wire Wire Line
 	8200 2300 7300 2300
 $Comp
-L R R6
+L Device:R R6
 U 1 1 5656453E
 P 8100 1750
@@
 Connection ~ 8100 2200
 $Comp
-L +3V3 #PWR017
+L power:+3V3 #PWR017
 U 1 1 5656523D
 P 8100 1550
@@
 	3950 1600 4300 1600
 Wire Wire Line
-	9150 5600 10550 5600
+	9150 5600 9450 5600
 Text Notes 1150 1000 1    60   ~ 0
 ON
@@
 BOOT0
 Wire Wire Line
-	2650 1100 1550 1100
+	2650 1100 2550 1100
 Wire Wire Line
 	2550 1150 2550 1100
 Connection ~ 2550 1100
 $Comp
-L +5V #PWR018
+L power:+5V #PWR018
 U 1 1 57F34D83
 P 900 1000
@@
 $EndComp
 Wire Wire Line
-	900  1000 900  1550
+	900  1000 900  1100
 Wire Wire Line
 	900  1550 1000 1550
@@
 	700  2050 700  700
 $Comp
-L STRIP_8P STRIP1
+L TCKB:STRIP_8P STRIP1
 U 1 1 57F7F91D
 P 10550 5200
@@
 NoConn ~ 4300 4200
 NoConn ~ 7300 2400
+Wire Wire Line
+	5650 4650 5800 4650
+Wire Wire Line
+	5800 4650 5950 4650
+Wire Wire Line
+	5950 1050 6100 1050
+Wire Wire Line
+	5800 1050 5950 1050
+Wire Wire Line
+	5650 1050 5800 1050
+Wire Wire Line
+	4100 6950 4100 7000
+Wire Wire Line
+	4100 6800 4100 6950
+Wire Wire Line
+	4350 6950 4500 6950
+Wire Wire Line
+	5800 6800 5800 7000
+Wire Wire Line
+	4100 7350 4100 7400
+Wire Wire Line
+	5800 7350 5800 7400
+Wire Wire Line
+	5550 6800 5800 6800
+Wire Wire Line
+	10400 1250 10700 1250
+Wire Wire Line
+	10100 1250 10400 1250
+Wire Wire Line
+	9800 1250 10100 1250
+Wire Wire Line
+	9800 850  10100 850
+Wire Wire Line
+	10100 850  10400 850
+Wire Wire Line
+	10400 850  10700 850
+Wire Wire Line
+	8950 3350 8950 3400
+Wire Wire Line
+	9200 3350 9300 3350
+Wire Wire Line
+	9300 3350 9400 3350
+Wire Wire Line
+	9400 3350 9500 3350
+Wire Wire Line
+	8100 2200 8200 2200
+Wire Wire Line
+	2550 1100 1550 1100
+Wire Wire Line
+	900  1400 900  1550
+Wire Wire Line
+	900  1250 900  1400
+Wire Wire Line
+	900  1100 900  1250
+Wire Wire Line
+	9450 5600 10550 5600
+Wire Wire Line
+	5950 4650 6100 4650
 $EndSCHEMATC
